File: kicad/_saved_ledcontroller.sch (KiCad schematic (older format))
At the start: 57 parts, among them J1 USB_A, J2 Pulse-J0026D21B, J3 STELVIO-2P-508, J4 STELVIO-2P-508, J5 STELVIO-5P-508, J6 STELVIO-4P-508, P1 FDI_Cable, P2 CONN_01X02, P3 CONN_01X02, P4 CONN_01X02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

Commit message: PCB: Basic placement and initial routing ok
Connections:
- net SENS_PWR: now reaches J6.1, P4.2 (P2), P5.1 (P1)
Changed lines of the file:
@@
 Text Label 6950 4650 0    60   ~ 0
 FET_PWR
+Text Label 3350 6350 0    60   ~ 0
+SENS_PWR
 $EndSCHEMATC
